File: egl/v0.9/v0.9.sch (EAGLE design)
At the start: 57 parts, among them IC1 74HC125N, IC2 TINY25, IC3 ATTINY2313, Q2 12Mhz, X2 USBB-G

Commit message: [work on eagle] Made the board a perfect fit in a 100x100mm square and made it ready for manufacturer production by grouping objects in appropriate layers.
Parts:
- removed LED5: Verde, led:LED3MM
- removed S4, S5: TACT-64N, switch-omron:10-XX
- added DZ1, DZ2: 3v3, diode:ZENER-DIODEZD-7.5
- added X1: 12Mhz, murata-resonators:CSTLS_X
- D1, D2: value 3v3 -> TACT-64N; device diode:ZENER-DIODEZD-7.5 -> switch-omron:10-XX
- Q2: value 12Mhz -> Verde; device murata-resonators:CSTLS_X -> led:LED3MM
- R22, R23, R7: device rcl:R-EU_0207/10 -> rcl:R-EU_0204/7
- renumbered LED10 to Q7, LED3 to Q0, LED4 to Q1, LED6 to Q3, LED7 to Q4, LED8 to Q5, LED9 to Q6, S10 to D7, S3 to D0, S6 to D3, S7 to D4, S8 to D5, S9 to D6
Connections:
- net GND: now also D1.S, D1.S1, D2.S, D2.S1, DZ1.A, DZ2.A, Q2.C, X1.VSS; no longer D1.A, D2.A, LED5.C, Q2.VSS, S4.S, S4.S1, S5.S, S5.S1
- net N$17: now also DZ2.C; no longer D2.C
- net N$18: now also X1.1; no longer Q2.1
- net N$19: now also DZ1.C; no longer D1.C
- net N$20: now also X1.3; no longer Q2.3
- net N$22: now also Q2.A; no longer LED5.A
- net N$36: now also D1.P, D1.P1; no longer S4.P, S4.P1
- net N$37: now also D2.P, D2.P1; no longer S5.P, S5.P1
